File: pcb/pcb_rev.1.3/Sidblaster TicTac - Rev.1.3.sch (EAGLE design)
At the start: 55 parts, among them J1 MONOSW2, J2 MONOSW2, T1 PN2222, U1 PIC16F886-I/SP, U2 FT232RL, U3 6581, U4 MT3608, X1 USB-B-H

Commit message: Rev.1.3 small fix
Other:
- note added: "1.3"
- note removed: "1.2"
Changed lines of the file:
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@@
  9V: Rx = 14k</text>
 <text x="119.38" y="60.96" size="1.778" layer="91">+9V when closed</text>
-<text x="378.46" y="7.62" size="2.54" layer="91" font="vector">1.2</text>
+<text x="378.46" y="7.62" size="2.54" layer="91" font="vector">1.3</text>
 <text x="292.1" y="27.94" size="2.54" layer="91" font="vector">www.crazy-midi.de</text>
 </plain>
