File: pcb/pcb_rev.1.4/Sidblaster TicTac - Rev.1.4.brd (EAGLE design)
At the start: 80 x 46 mm, 61 parts, among them J1 MONOSW2, J2 MONOSW2, Q1 IRLML6402TRPBF, T1 PN2222, U1 PIC16F886-I/SP, U2 FT232RL, U3 6581, U4 MT3608, X1 USB-B-H

Commit message: Rev. 1.4
Parts:
- C18: value 1000pF -> 1000 pF
- C70, C71: value 470pF -> 470 pF
- C72, C73: value 22nF -> 22 nF
- C77: value 1µF/10µF -> 1 µF/10 µF
- C79: value 1 µF/10µF -> 1 µF/10 µF
- C8, C9: value 100nF -> 100 nF
- C80, C81: value 1800pF -> 1800 pF
- C82, C83: value 2200pF -> 2200 pF
- F1: value Ferrit -> (none)
- JP1: value Voltage Select -> (none)
- JP2: value CAP2 -> (none)
- JP3: value CAP1 -> (none)
- JP4: value POTX -> (none)
- JP5: value POTY -> (none)
- JP6: value Shield2GND -> (none)
- R12, R8: value 1k -> 1 k
- R14, R9: value 10k -> 10 k
- R20, R21, R3, R4: value 1k -> 1K
- R22: value 47k -> 47K
- R23: value 18k -> 18K
- SV1: value ISP -> (none)
- SV2: value Paddles -> (none)
Connections:
- net N$28 renamed C1
- net PWRLED renamed N$28
- removed net PWREN: R3.1, R4.2, U2.14
- new net N$34: R3.1, R4.1, U2.14
- net VCC: now also R4.2; no longer R4.1
Routing:
- net N$34: track 0.00 -> 19.3 mm, vias 0 -> 2
- net PWREN: track 18.8 -> 0.00 mm, vias 2 -> 0
- net GND: track 229.1 -> 235.6 mm
- net C1: track 0.00 -> 3.20 mm
- net VCC: track 91.8 -> 94.5 mm
